File: KICAD_V2/Espruino_Harness_V2/routing_control.kicad_sch (KiCad schematic)
At the start: 0 parts

Commit message: Add V2 routing logic library prototypes
Parts:
- added IC1: MCP23017-E_SP, SamacSys_Parts:DIP794W56P254L3486H508Q28N, symbol SamacSys_Parts:MCP23017-E_SP
- added IC2: MCP23008-E_P, SamacSys_Parts:DIP794W56P254L2286H533Q18N, symbol SamacSys_Parts:MCP23008-E_P
- added Q1: DG409LEDY-GE3, SamacSys_Parts:SOIC127P600X175-16N, symbol V2_Harness:DG409LEDY-Multiplexer-Switch-Dual-4-Ch
- added R4: 470R, V2_Harness:R_Axial_DIN0204_L3.6mm_D1.6mm_P2.54mm_Vertical, symbol Device:R
- added SEL_D26: LOOP_B / DS2413_PIOB, V2_Harness:PinHeader_1x03_P2.54mm_Vertical, symbol Jumper:Jumper_3_Open
- added U3: TMUX1204DGSR, V2_Harness:SOIC_EDY-GE3_VIS, symbol V2_Harness:TMUX1204DGSR--4{colon}1-1-channel-analog-multiplexer
Connections:
- new net: R4.1, SEL_D26.2 (C)
- new net D25_LOOP_B_OUT: Q1.1 (A0), Q1.2 (EN), Q1.3 (V-), Q1.4 (S1A), Q1.5 (S2A), Q1.6 (S3A), Q1.7 (S4A), Q1.8 (DA), SEL_D26.1 (A)
- new net D26_LOOP_B_IN: R4.2
- new net DS2413_PIOB: SEL_D26.3 (B)
