File: KICAD_V2/Espruino_Harness_V2/routing_switches.kicad_sch (KiCad schematic)
At the start: 0 parts

Commit message: Add Espruino Pico castellated footprints
Parts:
- added U1: Espruino-Pico-1v4, V2_Targets:Espruino-Pico-1v4-Gordon-Shim, symbol V2_Targets:Espruino-Pico-1v4
Changed lines of the file:
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@@
 	(generator_version "9.0")
 	(paper "A4")
+	(symbol
+		(lib_id "V2_Targets:Espruino-Pico-1v4")
+		(at 119.38 74.93 0)
+		(unit 1)
+		(exclude_from_sim no)
+		(in_bom yes)
+		(on_board yes)
+		(dnp no)
+		(fields_autoplaced yes)
+		(property "Reference" "U1"
+			(at 119.38 49.53 0)
+			(effects
+				(font
+					(size 1.27 1.27)
+				)
+			)
+		)
+		(property "Value" "Espruino-Pico-1v4"
+			(at 119.38 52.07 0)
+			(effects
+				(font
+					(size 1.27 1.27)
+				)
+			)
+		)
+		(property "Footprint" "V2_Targets:Espruino-Pico-1v4-Gordon-Shim"
+			(at 119.38 74.93 0)
+			(effects
+				(font
+					(size 1.27 1.27)
+				)
+				(hide yes)
+			)
+		)
+		(property "Datasheet" ""
+			(at 119.38 74.93 0)
+			(effects
+				(font
+					(size 1.27 1.27)
+				)
+				(hide yes)
+			)
+		)
+		(property "Description" "V2 wirewrap target board"
+			(at 119.38 74.93 0)
+			(effects
+				(font
+					(size 1.27 1.27)
+				)
+				(hide yes)
+			)
+		)
+		(pin "A6"
+		)
+		(pin "B10"
+		)
+		(pin "B5"
+		)
+		(pin "B15"
+		)
+		(pin "B4"
+		)
+		(pin "5V"
+		)
+		(pin "B3"
+		)
+		(pin "B8"
+		)
+		(pin "A5"
+		)
+		(pin "A7"
+		)
+		(pin "VDD"
+		)
+		(pin "VBAT"
+		)
+		(pin "B1"
+		)
+		(pin "B14"
+		)
+		(pin "GND"
+		)
+		(pin "B9"
+		)
+		(pin "B13"
+		)
+		(pin "A8"
+		)
+		(pin "B6"
+		)
+		(pin "B7"
+		)
+		(pin "A10"
+		)
+		(pin "A1"
+		)
+		(pin "A2"
+		)
+		(pin "A0"
+		)
+		(pin "A3"
+		)
+		(pin "A4"
+		)
+		(instances
+			(project ""
+				(path "/d963e9d0-39be-47fe-b8bd-9ec6fa256faa/c2451a36-5070-407f-ac11-fc6972885dd1"
+					(reference "U1")
+					(unit 1)
+				)
+			)
+		)
+	)
 )
