File: KICAD_V2/Espruino_Harness_V2/target_interface.kicad_sch (KiCad schematic)
At the start: 7 parts, among them U1 Espruino-MDBT42Q-Breakout, U2 Espruino-Pico-1v4, U3 Raspberry-Pi-Pico-Family, U4 ESP32-S3-DevKitC-1, U5 OLIMEX-ESP32-S3-DevKit-LiPo-EA, U6 ESP32-DevKitC-V4, U7 ESP32-C3-DevKitC-02

Commit message: Add V2 routing logic library prototypes
Parts:
- removed U3: Raspberry-Pi-Pico-Family, V2_Targets:Raspberry-Pi-Pico-Family-Wirewrap, symbol V2_Targets:Raspberry-Pi-Pico-Family
Changed lines of the file:
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@@
 	(paper "A4")
-	(symbol
-		(lib_id "V2_Targets:Raspberry-Pi-Pico-Family")
-		(at 172.72 55.88 0)
-		(unit 1)
-		(exclude_from_sim no)
-		(in_bom yes)
-		(on_board yes)
-		(dnp no)
-		(fields_autoplaced yes)
-		(property "Reference" "U3"
-			(at 172.72 20.32 0)
-			(effects
-				(font
-					(size 1.27 1.27)
-				)
-			)
-		)
-		(property "Value" "Raspberry-Pi-Pico-Family"
-			(at 172.72 22.86 0)
-			(effects
-				(font
-					(size 1.27 1.27)
-				)
-			)
-		)
-		(property "Footprint" "V2_Targets:Raspberry-Pi-Pico-Family-Wirewrap"
-			(at 172.72 55.88 0)
-			(effects
-				(font
-					(size 1.27 1.27)
-				)
-				(hide yes)
-			)
-		)
-		(property "Datasheet" ""
-			(at 172.72 55.88 0)
-			(effects
-				(font
-					(size 1.27 1.27)
-				)
-				(hide yes)
-			)
-		)
-		(property "Description" "Provisional V2 target symbol"
-			(at 172.72 55.88 0)
-			(effects
-				(font
-					(size 1.27 1.27)
-				)
-				(hide yes)
-			)
-		)
-		(pin "4"
-		)
-		(pin "18"
-		)
-		(pin "20"
-		)
-		(pin "23"
-		)
-		(pin "2"
-		)
-		(pin "16"
-		)
-		(pin "27"
-		)
-		(pin "22"
-		)
-		(pin "1"
-		)
-		(pin "12"
-		)
-		(pin "5"
-		)
-		(pin "21"
-		)
-		(pin "10"
-		)
-		(pin "11"
-		)
-		(pin "8"
-		)
-		(pin "7"
-		)
-		(pin "3"
-		)
-		(pin "13"
-		)
-		(pin "9"
-		)
-		(pin "14"
-		)
-		(pin "6"
-		)
-		(pin "15"
-		)
-		(pin "17"
-		)
-		(pin "19"
-		)
-		(pin "24"
-		)
-		(pin "25"
-		)
-		(pin "26"
-		)
-		(pin "40"
-		)
-		(pin "29"
-		)
-		(pin "32"
-		)
-		(pin "36"
-		)
-		(pin "33"
-		)
-		(pin "37"
-		)
-		(pin "30"
-		)
-		(pin "31"
-		)
-		(pin "35"
-		)
-		(pin "38"
-		)
-		(pin "39"
-		)
-		(pin "28"
-		)
-		(pin "34"
-		)
-		(instances
-			(project ""
-				(path "/d963e9d0-39be-47fe-b8bd-9ec6fa256faa/6b2aa498-f7c9-4b40-a07e-030f921560ad"
-					(reference "U3")
-					(unit 1)
-				)
-			)
-		)
-	)
 	(symbol
 		(lib_id "V2_Targets:Espruino-MDBT42Q-Breakout")

Commit message: Add Espruino Pico castellated footprints
Parts:
- removed U1: Espruino-MDBT42Q-Breakout, V2_Targets:Espruino-MDBT42Q-Breakout-Wirewrap, symbol V2_Targets:Espruino-MDBT42Q-Breakout
- removed U2: Espruino-Pico-1v4, V2_Targets:Espruino-Pico-1v4-Wirewrap, symbol V2_Targets:Espruino-Pico-1v4
- removed U4: ESP32-S3-DevKitC-1, V2_Targets:ESP32-S3-DevKitC-1, symbol V2_Targets:ESP32-S3-DevKitC-1
- removed U5: OLIMEX-ESP32-S3-DevKit-LiPo-EA, V2_Targets:OLIMEX-ESP32-S3-DevKit-LiPo-EA-Wirewrap, symbol V2_Targets:OLIMEX-ESP32-S3-DevKit-LiPo-EA
- removed U6: ESP32-DevKitC-V4, V2_Targets:ESP32-DevKitC-V4-Wirewrap, symbol V2_Targets:ESP32-DevKitC-V4
- removed U7: ESP32-C3-DevKitC-02, V2_Targets:ESP32-C3-DevKitC-02, symbol V2_Targets:ESP32-C3-DevKitC-02
