File: KICAD/V2/RevA/Espruino_Harness_RevA/standard_test_blocks.kicad_sch (KiCad schematic)
At the start: 91 parts, among them J201 EXTERNAL_ANALOG_STIMULUS_0_TO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, J301 GROVE_I2C, J302 MCP23017_GPIO, J401 MCP3008_ANALOGUE_BREAKOUT, J402 PIHUT_MICROSD_BREAKOUT_106696, J501 DS18B20_SENSOR_A, J502 DS18B20_SENSOR_B, J503 2K2_DQ_4K7, J504 DS2413_MODULE, J701 UART_PEER_DIAGNOSTIC, J902 PIXEL_SHIFTER_6066, Q301 2N7002, Q302 2N7002, U301 MCP23017-E/SO, U401 MCP3008, U701 TMUX1511

Commit message: Establish Rev-A schematic verification framework
Changed lines of the file:
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@@
 	)
 	(junction
+		(at 121.92 134.62)
+		(diameter 0)
+		(color 0 0 0 0)
+	)
+	(junction
 		(at 454.66 73.66)
 		(diameter 0)
@@
 	(wire
 		(pts
+			(xy 121.92 134.62) (xy 121.92 138.43)
+		)
+		(stroke
+			(width 0)
+			(type default)
+		)
+	)
+	(wire
+		(pts
 			(xy 496.57 212.09) (xy 496.57 214.63)
 		)
@@
 	(wire
 		(pts
+			(xy 185.42 147.32) (xy 210.82 147.32)
+		)
+		(stroke
+			(width 0)
+			(type default)
+		)
+	)
+	(wire
+		(pts
 			(xy 408.94 43.18) (xy 430.53 43.18)
 		)
@@
 	(wire
 		(pts
-			(xy 392.43 295.91) (xy 402.59 295.91)
+			(xy 391.16 295.91) (xy 402.59 295.91)
 		)
 		(stroke
@@
 	(wire
 		(pts
+			(xy 115.57 134.62) (xy 121.92 134.62)
+		)
+		(stroke
+			(width 0)
+			(type default)
+		)
+	)
+	(wire
+		(pts
 			(xy 506.73 321.31) (xy 513.08 321.31)
 		)
@@
 	(wire
 		(pts
-			(xy 185.42 147.32) (xy 210.82 147.32)
-		)
-		(stroke
-			(width 0)
-			(type default)
-		)
-	)
-	(wire
-		(pts
 			(xy 396.24 215.9) (xy 396.24 218.44)
 		)
@@
 	(wire
 		(pts
-			(xy 121.92 127) (xy 121.92 138.43)
+			(xy 121.92 127) (xy 121.92 134.62)
 		)
 		(stroke
@@
 		)
 	)
-	(label "TI_ONEWIRE_DQ"
-		(at 392.43 295.91 180)
-		(effects
-			(font
-				(size 1.27 1.27)
-			)
-			(justify right bottom)
-		)
-	)
 	(label "TEST_BLOCK_3V3"
 		(at 392.43 298.45 180)
@@
 		)
 	)
+	(label "TI_ONEWIRE_DQ"
+		(at 391.16 295.91 180)
+		(effects
+			(font
+				(size 1.27 1.27)
+			)
+			(justify right bottom)
+		)
+	)
 	(label "ANALOG_FB"
 		(at 515.62 62.23 180)
@@
 	)
 	(hierarchical_label "TI_ONEWIRE_DQ"
-		(shape input)
+		(shape bidirectional)
 		(at 389.89 326.39 180)
 		(effects
@@
 			)
 		)
-		(property "Datasheet" "https://www.onsemi.com/pub/Collateral/NDS7002A-D.PDF"
+		(property "Datasheet" "https://assets.nexperia.com/documents/data-sheet/2N7002.pdf"
 			(at 411.48 215.9 0)
 			(effects
@@
 			)
 		)
-		(property "Description" "Protected Supervisor stimulus open-drain stage"
+		(property "Description" "2N7002 60 V N-channel enhancement MOSFET, pin 1 gate, pin 2 source, pin 3 drain, SOT-23"
 			(at 411.48 215.9 0)
 			(effects
@@
 	)
 	(symbol
+		(lib_id "power:PWR_FLAG")
+		(at 115.57 134.62 0)
+		(unit 1)
+		(exclude_from_sim no)
+		(in_bom yes)
+		(on_board yes)
+		(dnp no)
+		(fields_autoplaced yes)
+		(property "Reference" "#FLG06"
+			(at 115.57 132.715 0)
+			(effects
+				(font
+					(size 1.27 1.27)
+				)
+				(hide yes)
+			)
+		)
+		(property "Value" "PWR_FLAG"
+			(at 115.57 129.54 0)
+			(effects
+				(font
+					(size 1.27 1.27)
+				)
+			)
+		)
+		(property "Footprint" ""
+			(at 115.57 134.62 0)
+			(effects
+				(font
+					(size 1.27 1.27)
+				)
+				(hide yes)
+			)
+		)
+		(property "Datasheet" "~"
+			(at 115.57 134.62 0)
+			(effects
+				(font
+					(size 1.27 1.27)
+				)
+				(hide yes)
+			)
+		)
+		(property "Description" "Special symbol for telling ERC where power comes from"
+			(at 115.57 134.62 0)
+			(effects
+				(font
+					(size 1.27 1.27)
+				)
+				(hide yes)
+			)
+		)
+		(pin "1"
+		)
+		(instances
+			(project ""
+				(path "/12444148-a051-4fb0-ae7b-e3d34eecc954/de8f4588-cd43-45f8-a502-51219f80935f"
+					(reference "#FLG06")
+					(unit 1)
+				)
+			)
+		)
+	)
+	(symbol
 		(lib_id "Device:R")
 		(at 182.88 198.12 0)
@@
 	)
 	(symbol
+		(lib_name "NMOS_2N7002_GSD_1")
 		(lib_id "Espruino_Harness_RevA:NMOS_2N7002_GSD")
 		(at 511.81 212.09 0)
@@
 			)
 		)
-		(property "Datasheet" "https://www.onsemi.com/pub/Collateral/NDS7002A-D.PDF"
+		(property "Datasheet" "https://assets.nexperia.com/documents/data-sheet/2N7002.pdf"
 			(at 511.81 212.09 0)
 			(effects
@@
 			)
 		)
-		(property "Description" "Protected open-drain Supervisor acknowledgement stage"
+		(property "Description" "2N7002 60 V N-channel enhancement MOSFET, pin 1 gate, pin 2 source, pin 3 drain, SOT-23"
 			(at 511.81 212.09 0)
 			(effects
@@
 					(size 1.27 1.27)
 				)
+				(hide yes)
 			)
 		)
@@
 		(dnp no)
 		(property "Reference" "J503"
-			(at 425.45 323.85 90)
+			(at 426.72 323.85 90)
 			(effects
 				(font
@@
 		)
 		(property "Value" "2K2_DQ_4K7"
-			(at 429.26 327.66 90)
+			(at 430.53 326.39 90)
 			(effects
 				(font
