File: KICAD/V2/RevA/Espruino_Harness_RevA/power_control.kicad_sch (KiCad schematic)
At the start: 43 parts, among them J1001 OPERATING_MODE Selection, Q1001 DMN2024UQ-7, Q1101 AO3401A, U1001 TPS2116DRL, U1002 TPS22917DBV, U1101 TPS2559-Q1, U1102 TXU0101DBVR, U1103 INA226, U1104 INA228, U1105 74LVC2G08

Commit message: Verify Rev-A power control baseline
Other:
- note added: "TEST_BLOCK_SWITCH_EN high -> ROUTING_LOGIC_3V3 is passed to TEST_BLOCK_3V3 TEST_BLOCK_SWITCH_EN low -> TEST_BLOCK_3V3 is switched off and discharged"
- note added: "U1001 - TPS2116 Power Mux with Manual and Priority Switchover"
- note added: "U1001 - TPS22917 Ultra-Low Leakage Load Switch"
- note added: "U1001 selects the ROUTING_LOGIC_3V3 source: OFF -> output disabled STANDALONE -> TI_TARGET_3V3 STANDALONE EXT -> EXT_3V3 SUPERVISOR -> EXT_3V3"
- note added: "U1002 - TPS22917DBV Active-high Test Block 3.3 V load switch. C1005 controls turn-on slew and inrush current. QOD discharges TEST_BLOCK_3V3 when disabled. No current limiting or overload protection."
- note removed: "** Circuit Logic Sequence for operating mode and 3.3 V rails: D1001 MODE_EXT_SELECTED = MODE_STANDALONE_EXT OR MODE_SUPERVISOR D1002 MUX_MODE = MODE_STANDALONE OR MODE_EXT_SELECTED D1003 MODE_BIAS_3V3 = TI_TARGET_3V3 OR EXT_3V3 Diode-isolated logic bias only; it does not combine the load-power rails. Q1001 / R1002 MODE_EXT_SELECTED low -> MUX_PR1 high MODE_EXT_SELECTED high -> MUX_PR1 low U1001 s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"
- note removed: "TPS2116 Power Mux with Manual and Priority Switchover"
- note removed: "TPS22917 Ultra-Low Leakage Load Switch"
- note removed: "TPS22917DBV Active-high Test Block 3.3 V load switch. C1005 controls turn-on slew and inrush current. QOD discharges TEST_BLOCK_3V3 when disabled. No current limiting or overload protection."
- note removed: "| Device| OR inputs | Output | | |-------|---------------------------------------------|------------------------|-----------------------------------------------------------------------------------| | D1001 | `MODE_STANDALONE_EXT`, `MODE_SUPERVISOR` | `MODE_EXT_SELECTED` | Indicates that U1001 must use the external 3.3 V supply. | | D1002 | `MODE_STANDALONE`, `MODE_EXT_SELECTED` | `MUX_MODE` | Ena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"
Changed lines of the file:
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@@
 	)
 	(rectangle
-		(start 41.91 16.51)
-		(end 386.08 120.65)
+		(start 44.45 16.51)
+		(end 383.54 120.65)
 		(stroke
 			(width 0.254)
@@
 	)
 	(rectangle
-		(start 43.18 123.19)
-		(end 387.35 284.48)
+		(start 44.45 123.19)
+		(end 383.54 284.48)
 		(stroke
 			(width 0.254)
@@
 		)
 	)
-	(text "TPS2116\n Power Mux with Manual and Priority Switchover"
+	(text "U1001 - TPS2116\n Power Mux with Manual and Priority Switchover"
 		(exclude_from_sim no)
 		(at 300.99 95.25 0)
@@
 	(text "TARGET_POWER_FAULT_N asserts low on overcurrent or overtemperature."
 		(exclude_from_sim no)
-		(at 81.28 140.97 0)
+		(at 83.82 142.24 0)
 		(effects
 			(font
@@
 		)
 	)
-	(text "TPS22917DBV\nActive-high Test Block 3.3 V load switch.\nC1005 controls turn-on slew and inrush current.\nQOD discharges TEST_BLOCK_3V3 when disabled.\nNo current limiting or overload protection."
+	(text "U1002 - TPS22917DBV\n	Active-high Test Block 3.3 V load switch.\n	C1005 controls turn-on slew and inrush current.\n	QOD discharges TEST_BLOCK_3V3 when disabled.\n	No current limiting or overload protection."
 		(exclude_from_sim no)
-		(at 327.66 64.77 0)
-		(effects
-			(font
-				(size 1.27 1.27)
-			)
-			(justify left)
-		)
-	)
-	(text "** Circuit Logic Sequence for operating mode and 3.3 V rails:\n\nD1001\nMODE_EXT_SELECTED =\n    MODE_STANDALONE_EXT OR MODE_SUPERVISOR\n\nD1002\nMUX_MODE =\n    MODE_STANDALONE OR MODE_EXT_SELECTED\n\nD1003\nMODE_BIAS_3V3 =\n    TI_TARGET_3V3 OR EXT_3V3\nDiode-isolated logic bias only; it does not combine the load-power rails.\n\nQ1001 / R1002\nMODE_EXT_SELECTED low  -> MUX_PR1 high\nMODE_EXT_SELECTED high -> MUX_PR1 low\n\nU1001 selects the ROUTING_LOGIC_3V3 source:\nOFF               -> output disabled\nSTANDALONE        -> TI_TARGET_3V3\nSTANDALONE EXT    -> EXT_3V3\nSUPERVISOR        -> EXT_3V3\n\nD1004\nTEST_BLOCK_AUTO_EN =\n    MODE_STANDALONE OR MODE_STANDALONE_EXT\n\nD1005\nTEST_BLOCK_SWITCH_EN =\n    TEST_BLOCK_AUTO_EN OR TEST_BLOCK_POWER_EN\n\nU1002\nTEST_BLOCK_SWITCH_EN high\n    -> ROUTING_LOGIC_3V3 is passed to TEST_BLOCK_3V3\n\nTEST_BLOCK_SWITCH_EN low\n    -> TEST_BLOCK_3V3 is switched off and discharged"
-		(exclude_from_sim no)
-		(at -60.96 48.26 0)
+		(at 318.77 64.77 0)
 		(effects
 			(font
@@
 		)
 	)
-	(text "| Device| OR inputs                                   |       Output           |                                                                                   |                             \n|-------|---------------------------------------------|------------------------|-----------------------------------------------------------------------------------|\n| D1001 | `MODE_STANDALONE_EXT`, `MODE_SUPERVISOR`    | `MODE_EXT_SELECTED`    | Indicates that U1001 must use the external 3.3 V supply.                          |\n| D1002 | `MODE_STANDALONE`, `MODE_EXT_SELECTED`      | `MUX_MODE`             | Enables U1001 in every active operating mode; remains low in OFF                  |\n| D1003 | `TI_TARGET_3V3`, `EXT_3V3`                  | `MODE_BIAS_3V3`        | Supplies the low-current bias used to establish U1001's source-selection state.   |\n| D1004 | `MODE_STANDALONE`, `MODE_STANDALONE_EXT`    | `TEST_BLOCK_AUTO_EN`   | Automatically requests Test Block power in either standalone mode.                |\n| D1005 | `TEST_BLOCK_AUTO_EN`, `TEST_BLOCK_POWER_EN` | `TEST_BLOCK_SWITCH_EN` | Enables U1002 from either the standalone automatic request or Supervisor command. |"
-		(exclude_from_sim no)
-		(at -331.47 153.67 0)
-		(effects
-			(font
-				(face "Consolas")
-				(size 1.524 1.524)
-			)
-			(justify left)
-		)
-	)
 	(text "SUPERVISOR"
 		(exclude_from_sim no)
@@
 	(text "TARGET 5 V SWITCH AND TWO-RANGE POWER MONITOR"
 		(exclude_from_sim no)
-		(at 44.45 128.27 0)
+		(at 46.99 128.27 0)
 		(effects
 			(font
@@
 		)
 	)
-	(text "TPS22917\nUltra-Low Leakage Load Switch"
+	(text "TEST_BLOCK_SWITCH_EN high\n    -> ROUTING_LOGIC_3V3 is passed to TEST_BLOCK_3V3\n\nTEST_BLOCK_SWITCH_EN low\n    -> TEST_BLOCK_3V3 is switched off and discharged"
 		(exclude_from_sim no)
-		(at 354.33 95.25 0)
+		(at 323.85 77.47 0)
+		(effects
+			(font
+				(size 1.27 1.27)
+			)
+			(justify left)
+		)
+	)
+	(text "U1001 - TPS22917\nUltra-Low Leakage Load Switch"
+		(exclude_from_sim no)
+		(at 351.79 95.25 0)
 		(effects
 			(font
@@
 	(text "In Supervisor mode, this block switches EXT_5V to the target with controlled turn-on,\nresistor-programmed current limiting, fault reporting, and normal or sleep-current measurement.\n\nThe normal/high-current measurement range is the hardware-safe default.\nReverse-current blocking while disabled permits independent Standalone target power."
 		(exclude_from_sim no)
-		(at 45.72 134.62 0)
+		(at 48.26 134.62 0)
+		(effects
+			(font
+				(size 1.27 1.27)
+			)
+			(justify left)
+		)
+	)
+	(text "U1001 \nselects the ROUTING_LOGIC_3V3 source:\n	OFF               -> output disabled\n	STANDALONE        -> TI_TARGET_3V3\n	STANDALONE EXT    -> EXT_3V3\n	SUPERVISOR        -> EXT_3V3\n"
+		(exclude_from_sim no)
+		(at 247.65 105.41 0)
 		(effects
 			(font
@@
 	(wire
 		(pts
-			(xy 354.33 38.1) (xy 365.76 38.1)
+			(xy 354.33 38.1) (xy 363.22 38.1)
 		)
 		(stroke
@@
 	)
 	(image
-		(at 369.57 107.95)
+		(at 367.03 107.95)
 		(scale 0.643104)
 		(data "iVBORw0KGgoAAAANSUhEUgAAAgEAAAGMCAYAAABDIHH6AAAABHNCSVQICAgIfAhkiAAAIABJREFU"
@@
 	(hierarchical_label "TEST_BLOCK_3V3"
 		(shape output)
-		(at 365.76 38.1 0)
+		(at 363.22 38.1 0)
 		(effects
 			(font

Commit message: Implement RC01 routing baseline metadata
Parts:
- C1102, C1103, C1104, C1105, C1106, C1107: AISLER_MPN (none) -> 100nF 10% 16V X7R 0603
- R1001, R1003, R1004, R1009, R1103, R1104, R1106, R1107, R1110: AISLER_MPN (none) -> 100k 0603 1% 0.1W
Changed lines of the file:
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@@
 			)
 		)
+		(property "AISLER_MPN" "100k 0603 1% 0.1W"
+			(at 167.64 256.54 90)
+			(effects
+				(font
+					(size 1.27 1.27)
+				)
+			)
+		)
 		(pin "1"
 		)
@@
 			)
 		)
+		(property "AISLER_MPN" "100nF 10% 16V X7R 0603"
+			(at 151.13 172.72 0)
+			(effects
+				(font
+					(size 1.27 1.27)
+				)
+			)
+		)
 		(pin "1"
 		)
@@
 			)
 		)
+		(property "AISLER_MPN" "100k 0603 1% 0.1W"
+			(at 74.93 255.27 90)
+			(effects
+				(font
+					(size 1.27 1.27)
+				)
+			)
+		)
 		(pin "1"
 		)
@@
 			)
 		)
+		(property "AISLER_MPN" "100nF 10% 16V X7R 0603"
+			(at 110.49 227.33 0)
+			(effects
+				(font
+					(size 1.27 1.27)
+				)
+			)
+		)
 		(pin "1"
 		)
@@
 			)
 		)
+		(property "AISLER_MPN" "100nF 10% 16V X7R 0603"
+			(at 189.23 186.69 0)
+			(effects
+				(font
+					(size 1.27 1.27)
+				)
+			)
+		)
 		(pin "1"
 		)
@@
 			)
 		)
+		(property "AISLER_MPN" "100k 0603 1% 0.1W"
+			(at 224.79 54.61 90)
+			(effects
+				(font
+					(size 1.27 1.27)
+				)
+			)
+		)
 		(pin "1"
 		)
@@
 			)
 		)
+		(property "AISLER_MPN" "100k 0603 1% 0.1W"
+			(at 208.28 254 90)
+			(effects
+				(font
+					(size 1.27 1.27)
+				)
+			)
+		)
 		(pin "1"
 		)
@@
 			)
 		)
+		(property "AISLER_MPN" "100k 0603 1% 0.1W"
+			(at 82.55 255.27 90)
+			(effects
+				(font
+					(size 1.27 1.27)
+				)
+			)
+		)
 		(pin "1"
 		)
@@
 			)
 		)
+		(property "AISLER_MPN" "100k 0603 1% 0.1W"
+			(at 86.36 175.26 0)
+			(effects
+				(font
+					(size 1.27 1.27)
+				)
+			)
+		)
 		(pin "1"
 		)
@@
 			)
 		)
+		(property "AISLER_MPN" "100nF 10% 16V X7R 0603"
+			(at 292.1 189.23 0)
+			(effects
+				(font
+					(size 1.27 1.27)
+				)
+			)
+		)
 		(pin "1"
 		)
@@
 			)
 		)
+		(property "AISLER_MPN" "100k 0603 1% 0.1W"
+			(at 177.8 53.34 90)
+			(effects
+				(font
+					(size 1.27 1.27)
+				)
+			)
+		)
 		(pin "1"
 		)
@@
 			)
 		)
+		(property "AISLER_MPN" "100nF 10% 16V X7R 0603"
+			(at 168.91 237.49 0)
+			(effects
+				(font
+					(size 1.27 1.27)
+				)
+			)
+		)
 		(pin "1"
 		)
@@
 			)
 		)
+		(property "AISLER_MPN" "100k 0603 1% 0.1W"
+			(at 90.17 255.27 90)
+			(effects
+				(font
+					(size 1.27 1.27)
+				)
+			)
+		)
 		(pin "1"
 		)
@@
 			)
 		)
+		(property "AISLER_MPN" "100k 0603 1% 0.1W"
+			(at 313.69 46.99 90)
+			(effects
+				(font
+					(size 1.27 1.27)
+				)
+			)
+		)
 		(pin "1"
 		)
@@
 			)
 		)
+		(property "AISLER_MPN" "100nF 10% 16V X7R 0603"
+			(at 208.28 237.49 0)
+			(effects
+				(font
+					(size 1.27 1.27)
+				)
+			)
+		)
