File: KICAD/V2/RevA/Espruino_Harness_RevA/power_control.kicad_sch (KiCad schematic)
At the start: 43 parts, among them J1001 OPERATING_MODE Selection, Q1001 DMN2024UQ-7, Q1101 AO3401A, U1001 TPS2116DRL, U1002 TPS22917DBV, U1101 TPS2559-Q1, U1102 TXU0101DBVR, U1103 INA226, U1104 INA228, U1105 74LVC2G08

Commit message: Verify TB03 I2C functional device baseline
Parts:
- R1101: footprint Espruino_Harness_RevA:R_Shunt_Yageo_PE2512_CurrentSense -> Resistor_SMD:R_0603_1608Metric
- R1102: footprint Espruino_Harness_RevA:R_Shunt_Bourns_CHP2512_CurrentSense -> Resistor_SMD:R_0603_1608Metric
Changed lines of the file:
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@@
 	)
 	(symbol
-		(lib_name "TI_GND_3")
 		(lib_id "Espruino_Harness_RevA:TI_GND")
 		(at 189.23 190.5 0)
@@
 	)
 	(symbol
-		(lib_name "C_7")
 		(lib_id "Espruino_Harness_RevA:C")
 		(at 276.86 46.99 180)
@@
 	)
 	(symbol
-		(lib_name "TI_GND_3")
 		(lib_id "Espruino_Harness_RevA:TI_GND")
 		(at 292.1 193.04 0)
@@
 	)
 	(symbol
-		(lib_name "TI_GND_1")
 		(lib_id "Espruino_Harness_RevA:TI_GND")
 		(at 151.13 175.26 0)
@@
 	)
 	(symbol
-		(lib_name "TI_GND_3")
 		(lib_id "Espruino_Harness_RevA:TI_GND")
 		(at 208.28 241.3 0)
@@
 	)
 	(symbol
-		(lib_name "TI_GND_3")
 		(lib_id "Espruino_Harness_RevA:TI_GND")
 		(at 110.49 232.41 0)
@@
 	)
 	(symbol
-		(lib_name "R_1")
 		(lib_id "Espruino_Harness_RevA:R")
 		(at 173.99 160.02 90)
@@
 			)
 		)
-		(property "Footprint" "Espruino_Harness_RevA:R_Shunt_Yageo_PE2512_CurrentSense"
+		(property "Footprint" "Resistor_SMD:R_0603_1608Metric"
 			(at 173.99 160.02 0)
 			(effects
@@
 			)
 		)
-		(property "Datasheet" "https://yageogroup.com/content/Resource%20Library/Datasheet/PYU-PE_521_ROHS_L.pdf"
+		(property "Datasheet" "~"
 			(at 173.99 160.02 0)
 			(effects
@@
 			)
 		)
-		(property "Description" "Yageo PE2512FKF7W0R05L, 50 mΩ, 1%, 100 ppm/°C, 2 W."
+		(property "Description" "Resistor"
 			(at 173.99 160.02 0)
 			(effects
@@
 	)
 	(symbol
-		(lib_name "TI_GND_6")
 		(lib_id "Espruino_Harness_RevA:TI_GND")
 		(at 354.33 52.07 0)
@@
 	)
 	(symbol
-		(lib_name "TI_GND_3")
 		(lib_id "Espruino_Harness_RevA:TI_GND")
 		(at 120.65 264.16 0)
@@
 	)
 	(symbol
-		(lib_name "TI_GND_3")
 		(lib_id "Espruino_Harness_RevA:TI_GND")
 		(at 341.63 201.93 0)
@@
 	)
 	(symbol
-		(lib_name "R_4")
 		(lib_id "Espruino_Harness_RevA:R")
 		(at 113.03 175.26 0)
@@
 	)
 	(symbol
-		(lib_name "BAT54C_AAK_3")
 		(lib_id "Espruino_Harness_RevA:BAT54C_AAK")
 		(at 156.21 49.53 0)
@@
 			)
 		)
-		(property "Datasheet" "https://www.vishay.com/docs/86410/bat54_bat54a_bat54c_bat54s.pdf"
+		(property "Datasheet" "https://assets.nexperia.com/documents/data-sheet/BAT54C.pdf"
 			(at 156.21 49.53 0)
 			(effects
@@
 			)
 		)
-		(property "Description" "Vishay BAT54C-E3-08 dual Schottky diode, common cathode pin 3, SOT-23"
+		(property "Description" "BAT54C dual Schottky diode, common cathode pin 3, SOT-23"
 			(at 156.21 49.53 0)
 			(effects
@@
 	)
 	(symbol
-		(lib_name "R_4")
 		(lib_id "Espruino_Harness_RevA:R")
 		(at 167.64 146.05 0)
@@
 	)
 	(symbol
-		(lib_name "TI_GND_3")
 		(lib_id "Espruino_Harness_RevA:TI_GND")
 		(at 302.26 220.98 0)
@@
 	)
 	(symbol
-		(lib_name "TI_GND_10")
 		(lib_id "Espruino_Harness_RevA:TI_GND")
 		(at 276.86 60.96 0)
@@
 	)
 	(symbol
-		(lib_name "R_9")
 		(lib_id "Espruino_Harness_RevA:R")
 		(at 167.64 256.54 0)
@@
 	)
 	(symbol
-		(lib_name "TI_GND_4")
 		(lib_id "Espruino_Harness_RevA:TI_GND")
 		(at 313.69 52.07 0)
@@
 	)
 	(symbol
-		(lib_name "C_6")
 		(lib_id "Espruino_Harness_RevA:C")
 		(at 245.11 57.15 180)
@@
 	)
 	(symbol
-		(lib_name "TI_GND_5")
 		(lib_id "Espruino_Harness_RevA:TI_GND")
 		(at 336.55 52.07 0)
@@
 	)
 	(symbol
-		(lib_name "R_2")
 		(lib_id "Espruino_Harness_RevA:R")
 		(at 215.9 146.05 90)
@@
 			)
 		)
-		(property "Footprint" "Espruino_Harness_RevA:R_Shunt_Bourns_CHP2512_CurrentSense"
+		(property "Footprint" "Resistor_SMD:R_0603_1608Metric"
 			(at 215.9 146.05 0)
 			(effects
@@
 			)
 		)
-		(property "Datasheet" "https://www.bourns.com/docs/product-datasheets/chp.pdf"
+		(property "Datasheet" "~"
 			(at 215.9 146.05 0)
 			(effects
@@
 			)
 		)
-		(property "Description" "Bourns CHP2512-FX-1R00ELF, 1 Ω, 1%, 100 ppm/°C, 3 W."
+		(property "Description" "Resistor"
 			(at 215.9 146.05 0)
 			(effects
@@
 	)
 	(symbol
-		(lib_name "R_3")
 		(lib_id "Espruino_Harness_RevA:R")
 		(at 243.84 200.66 0)
@@
 	)
 	(symbol
-		(lib_name "C_1")
 		(lib_id "Espruino_Harness_RevA:C")
 		(at 151.13 172.72 0)
@@
 	)
 	(symbol
-		(lib_name "TI_GND_3")
 		(lib_id "Espruino_Harness_RevA:TI_GND")
 		(at 226.06 198.12 0)
@@
 			)
 		)
-		(property "Datasheet" "https://www.vishay.com/docs/86410/bat54_bat54a_bat54c_bat54s.pdf"
+		(property "Datasheet" "https://assets.nexperia.com/documents/data-sheet/BAT54C.pdf"
 			(at 289.56 87.63 0)
 			(effects
@@
 			)
 		)
-		(property "Description" "Vishay BAT54C-E3-08 dual Schottky diode, common cathode pin 3, SOT-23"
+		(property "Description" "BAT54C dual Schottky diode, common cathode pin 3, SOT-23"
 			(at 289.56 87.63 0)
 			(effects
@@
 	)
 	(symbol
-		(lib_name "R_5")
 		(lib_id "Espruino_Harness_RevA:R")
 		(at 74.93 255.27 0)
@@
 	)
 	(symbol
-		(lib_name "C_4")
 		(lib_id "Espruino_Harness_RevA:C")
 		(at 110.49 227.33 0)
@@
 	)
 	(symbol
-		(lib_name "C_4")
 		(lib_id "Espruino_Harness_RevA:C")
 		(at 189.23 186.69 0)
@@
 	)
 	(symbol
-		(lib_name "BAT54C_AAK_1")
 		(lib_id "Espruino_Harness_RevA:BAT54C_AAK")
 		(at 156.21 30.48 0)
@@
 			)
 		)
-		(property "Datasheet" "https://www.vishay.com/docs/86410/bat54_bat54a_bat54c_bat54s.pdf"
+		(property "Datasheet" "https://assets.nexperia.com/documents/data-sheet/BAT54C.pdf"
 			(at 156.21 30.48 0)
 			(effects
@@
 			)
 		)
-		(property "Description" "Vishay BAT54C-E3-08 dual Schottky diode, common cathode pin 3, SOT-23"
+		(property "Description" "BAT54C dual Schottky diode, common cathode pin 3, SOT-23"
 			(at 156.21 30.48 0)
 			(effects
@@
 	)
 	(symbol
-		(lib_name "BAT54C_AAK_2")
 		(lib_id "Espruino_Harness_RevA:BAT54C_AAK")
 		(at 196.85 76.2 0)
@@
 			)
 		)
-		(property "Datasheet" "https://www.vishay.com/docs/86410/bat54_bat54a_bat54c_bat54s.pdf"
+		(property "Datasheet" "https://assets.nexperia.com/documents/data-sheet/BAT54C.pdf"
 			(at 196.85 76.2 0)
 			(effects
@@
 			)
 		)
-		(property "Description" "Vishay BAT54C-E3-08 dual Schottky diode, common cathode pin 3, SOT-23"
+		(property "Description" "BAT54C dual Schottky diode, common cathode pin 3, SOT-23"
 			(at 196.85 76.2 0)
 			(effects
@@
 	)
 	(symbol
-		(lib_name "TI_GND_2")
 		(lib_id "Espruino_Harness_RevA:TI_GND")
 		(at 95.25 151.13 0)
@@
 	)
 	(symbol
-		(lib_name "R_10")
 		(lib_id "Espruino_Harness_RevA:R")
 		(at 224.79 54.61 0)
@@
 	)
 	(symbol
-		(lib_name "R_8")
 		(lib_id "Espruino_Harness_RevA:R")
 		(at 208.28 254 0)
@@
 	)
 	(symbol
-		(lib_name "TI_GND_11")
 		(lib_id "Espruino_Harness_RevA:TI_GND")
 		(at 238.76 34.29 0)
@@
 	)
 	(symbol
-		(lib_name "TI_GND_13")
 		(lib_id "Espruino_Harness_RevA:TI_GND")
 		(at 195.58 57.15 0)
@@
 	)
 	(symbol
-		(lib_name "R_6")
 		(lib_id "Espruino_Harness_RevA:R")
 		(at 82.55 255.27 0)
@@
 	)
 	(symbol
-		(lib_name "R_4")
 		(lib_id "Espruino_Harness_RevA:R")
 		(at 86.36 175.26 0)
@@
 	)
 	(symbol
-		(lib_name "C_3")
 		(lib_id "Espruino_Harness_RevA:C")
 		(at 292.1 189.23 0)
@@
 	)
 	(symbol
-		(lib_name "TI_GND_3")
 		(lib_id "Espruino_Harness_RevA:TI_GND")
 		(at 193.04 264.16 0)
@@
 	)
 	(symbol
-		(lib_name "TI_GND_3")
 		(lib_id "Espruino_Harness_RevA:TI_GND")
 		(at 132.08 184.15 0)
@@
 	)
 	(symbol
-		(lib_name "TI_GND_3")
 		(lib_id "Espruino_Harness_RevA:TI_GND")
 		(at 200.66 218.44 0)
@@
 	)
 	(symbol
-		(lib_name "TI_GND_7")
 		(lib_id "Espruino_Harness_RevA:TI_GND")
 		(at 245.11 60.96 0)
@@
 			)
 		)
-		(property "Datasheet" "https://www.vishay.com/docs/86410/bat54_bat54a_bat54c_bat54s.pdf"
+		(property "Datasheet" "https://assets.nexperia.com/documents/data-sheet/BAT54C.pdf"
 			(at 243.84 90.17 0)
 			(effects
@@
 			)
 		)
-		(property "Description" "Vishay BAT54C-E3-08 dual Schottky diode, common cathode pin 3, SOT-23"
+		(property "Description" "BAT54C dual Schottky diode, common cathode pin 3, SOT-23"
 			(at 243.84 90.17 0)
 			(effects
@@
 	)
 	(symbol
-		(lib_name "R_11")
 		(lib_id "Espruino_Harness_RevA:R")
 		(at 177.8 53.34 0)
@@
 	)
 	(symbol
-		(lib_name "C_7")
 		(lib_id "Espruino_Harness_RevA:C")
 		(at 289.56 45.72 180)
@@
 			)
 		)
-		(property "Description" "TPS22917 CT timing capacitor for Test Block inrush control"
+		(property "Description" "TPS2116 VIN1 local input capacitor"
 			(at 289.56 45.72 0)
 			(effects
@@
 	)
 	(symbol
-		(lib_name "C_5")
 		(lib_id "Espruino_Harness_RevA:C")
 		(at 168.91 237.49 0)
@@
 			)
 		)
-		(property "Description" "TXU0101 VCCA 3.3 V decoupling"
+		(property "Description" "TPS2116 VIN1 local input capacitor"
 			(at 168.91 237.49 0)
 			(effects
@@
 	)
 	(symbol
-		(lib_name "R_7")
 		(lib_id "Espruino_Harness_RevA:R")
 		(at 90.17 255.27 0)
@@
 	)
 	(symbol
-		(lib_name "R_4")
 		(lib_id "Espruino_Harness_RevA:R")
 		(at 350.52 204.47 0)
@@
 	)
 	(symbol
-		(lib_name "C_2")
 		(lib_id "Espruino_Harness_RevA:C")
 		(at 95.25 148.59 0)
@@
 	)
 	(symbol
-		(lib_name "TI_GND_9")
 		(lib_id "Espruino_Harness_RevA:TI_GND")
 		(at 257.81 60.96 0)
@@
 	)
 	(symbol
-		(lib_name "TI_GND_3")
 		(lib_id "Espruino_Harness_RevA:TI_GND")
 		(at 168.91 241.3 0)
@@
 	)
 	(symbol
-		(lib_name "TI_GND_8")
 		(lib_id "Espruino_Harness_RevA:TI_GND")
 		(at 224.79 60.96 0)
@@
 	)
 	(symbol
-		(lib_name "C_5")
 		(lib_id "Espruino_Harness_RevA:C")
 		(at 208.28 237.49 0)
@@
 			)
 		)
-		(property "Description" "TXU0101 VCCB 5 V decoupling"
+		(property "Description" "TPS2116 VIN1 local input capacitor"
 			(at 208.28 237.49 0)
 			(effects
@@
 	)
 	(symbol
-		(lib_name "TI_GND_12")
 		(lib_id "Espruino_Harness_RevA:TI_GND")
 		(at 177.8 57.15 0)

Commit message: Correct Rev-A operating-mode power architecture
Parts:
- removed D1001, D1002, D1003, D1004: BAT54C-E3-08, Package_TO_SOT_SMD:SOT-23, symbol Espruino_Harness_RevA:BAT54C_AAK
- removed J1001: OPERATING_MODE Selection, Connector_PinHeader_2.54mm:PinHeader_2x04_P2.54mm_Vertical, symbol Espruino_Harness_RevA:Operating_Mode_2x04
- removed Q1001: DMN2024UQ-7, Package_TO_SOT_SMD:SOT-23, symbol Espruino_Harness_RevA:DMN2024UQ-7
- removed U1001: TPS2116DRL, Package_TO_SOT_SMD:SOT-583-8, symbol Espruino_Harness_RevA:TPS2116DRL_POWER_MUX
- added C1006: 470 pF, Capacitor_SMD:C_0603_1608Metric, symbol Espruino_Harness_RevA:C
- added C1007: 100 nF, Capacitor_SMD:C_0603_1608Metric, symbol Espruino_Harness_RevA:C
- added J1001: OPERATING MODE - 3V3 SOURCE, Connector_PinHeader_2.54mm:PinHeader_2x03_P2.54mm_Vertical, symbol Connector_Generic:Conn_02x03_Odd_Even
- added R1005: 249k, Resistor_SMD:R_0603_1608Metric, symbol Espruino_Harness_RevA:R
- added U1001: TPSM828438, symbol Espruino_Harness_RevA:TPSM828438_VCF_REGULATOR
- added U1003: TPS22917DBVR, Package_TO_SOT_SMD:SOT-23-6, symbol Espruino_Harness_RevA:TPS22917DBV_LOAD_SWITCH
- added U1004: SN74LVC2G14DBV, Package_TO_SOT_SMD:SOT-23-6, symbol 74xGxx:SN74LVC2G14DBV
- C1001: value 1uF -> 1 µF; AISLER_MPN (none) -> 1uF 10% 10V X7R 0603
- C1002: value 1uF -> 4.7 µF; footprint Capacitor_SMD:C_0603_1608Metric -> Capacitor_SMD:C_0805_2012Metric; AISLER_MPN (none) -> 4.7uF 10% 10V X7R 0805
- C1003: value 1uF -> 10 µF; footprint Capacitor_SMD:C_0603_1608Metric -> Capacitor_SMD:C_0805_2012Metric; AISLER_MPN (none) -> 10uF 10% 10V X7R 0805
- R1001: value 100k -> 10k; AISLER_MPN 100k 0603 1% 0.1W -> 10k 1% 0.1W 0603
- R1002: AISLER_MPN (none) -> 10k 1% 0.1W 0603
- R1003: value 100k -> 22k; AISLER_MPN 100k 0603 1% 0.1W -> 22k 1% 0.1W 0603
- R1004, R1009: value 100k -> 22k
Connections:
- net MUX_PR1 is gone; now on net TI_GND: R1002.2
- net TI_TARGET_3V3 is gone; now on net TI_GND: C1001.2
- net EXT_3V3: now also J1001.5 (Pin_5); no longer C1002.2
- net MODE_SUPERVISOR: now also U1004.3 (2A), U1004.6 (1Y)
- net ROUTING_LOGIC_3V3: now also C1007.1, J1001.3 (Pin_3), U1004.5 (V_{CC}); no longer C1003.2
- net TEST_BLOCK_AUTO_EN: now also U1004.4 (2Y)
- net TI_GND: now also C1002.2, C1003.2, C1007.2, R1005.1, U1001.1 (GND), U1003.2 (GND), U1004.2 (GND); no longer C1001.1, C1002.1, C1003.1, R1001.2
- net MODE_BIAS_3V3: no longer names the net of R1002.1
- net MODE_BIAS_3V3: now also J1001.6 (Pin_6)
- net MODE_EXT_SELECTED renamed LOCAL_REG_ENABLE
- net LOCAL_REG_ENABLE: now also J1001.4 (Pin_4), U1003.3 (ON), U1004.1 (1A)
- net MUX_MODE renamed TI_TARGET_VBUS
- net TI_TARGET_VBUS: now also C1001.1, C1006.2, U1003.1 (VIN)
- new net: C1006.1, U1003.4 (CT)
- new net: R1005.2, U1001.3 (VSET)
- new net: J1001.2 (Pin_2), R1001.2
- new net LOCAL_3V3: C1003.1, J1001.1 (Pin_1), U1001.6 (VOUT), U1001.7 (VOS)
- new net LOCAL_REG_VIN: C1002.1, U1001.2 (VIN), U1001.4 (EN), U1003.5 (QOD), U1003.6 (VOUT)
- no-connect marks 3 -> 1
Other:
- note added: "FUNCTIONAL FLOW Standalone: TI_TARGET_VBUS → U1003 isolation → U1001 regulator → LOCAL_3V3 → J1001 → ROUTING_LOGIC_3V3. U1004 asserts TEST_BLOCK_AUTO_EN; D1005 enables U1002. Supervisor: EXT_3V3 → J1001 → ROUTING_LOGIC_3V3. U1003 isolates and discharges LOCAL_REG_VIN; U1001 remains disabled. D1005 passes TEST_BLOCK_POWER_EN to U1002."
- note added: "Note LoopBack from Pin 6"
- note added: "OPERATING MODE — FIT TWO SHUNTS; CHANGE ONLY WHILE UNPOWERED Mode J1001 shunts Routing source Local regulator Test Block supply Standalone 1–3 and 2–4 LOCAL_3V3 Enabled Automatic Supervisor 3–5 and 4–6 EXT_3V3 Disabled/isolated TEST_BLOCK_POWER_EN"
- note added: "PCB-CRITICAL PLACEMENT Place C1001 and C1006 at U1003; C1002, C1003 and R1005 at U1001; C1007 directly at U1004 pins 5 and 2; and C1005/C1004 at U1002. Keep regulator power loops, CT connections and QOD discharge paths short."
- note added: "ROUTING_LOGIC_3V3"
- note added: "SAFE STATE R1003 holds LOCAL_REG_ENABLE low. R1009 holds MODE_SUPERVISOR low while its driver is unpowered. R1004 holds U1002 disabled. U1003 discharges LOCAL_REG_VIN and U1002 discharges TEST_BLOCK_3V3 when disabled."
- note added: "Selects LOCAL_3V3 or EXT_3V3 as the ROUTING_LOGIC_3V3 source. Derives the operating-mode state and controls automatic or Supervisor-commanded TEST_BLOCK_3V3."
- note added: "U1002 — TPS22917DBVR TEST-BLOCK LOAD SWITCH C1005 controls turn-on slew and inrush. QOD tied to VOUT discharges TEST_BLOCK_3V3 when disabled. No current limiting or overload protection is provided."
- note added: "U1003: C1006 = 470 pF from CT to VIN gives approximately 1.9 ms turn-on and about 23 mA initial charging current into C1002, typical. QOD is tied to VOUT for controlled LOCAL_REG_VIN discharge."
- note removed: "BAT54C diode ORs prevent the selected mode and source rails from backfeeding each other"
- note removed: "J1001 OFF: MODE low, PR1 high -> high-impedance output STANDALONE: MODE high, PR1 high -> TI_TARGET_3V3 STANDALONE EXT / SUPERVISOR: MODE high, PR1 low -> EXT_3V3 Change the Operating Mode shunt only with both 3.3 V sources off."
- note removed: "MODE_EXT_SELECTED"
- note removed: "MODE_STANDALONE"
- note removed: "MODE_STANDALONE_EXT"
- note removed: "MUX_MODE"
- note removed: "OFF"
- note removed: "R1001, R1003 and R1004 hold MODE, the inverter gate and Test Block enable low when undriven"
- note removed: "STANDALONE"
- note removed: "STANDALONE EXT"
- note removed: "SUPERVISOR"
- note removed: "Selects which 3.3 V source supplies ROUTING_LOGIC_3V3. Determines if that rail is passed on to TEST_BLOCK_3V3."
- note removed: "TEST_BLOCK_SWITCH_EN"
- note removed: "TEST_BLOCK_SWITCH_EN high -> ROUTING_LOGIC_3V3 is passed to TEST_BLOCK_3V3 TEST_BLOCK_SWITCH_EN low -> TEST_BLOCK_3V3 is switched off and discharged"
- note removed: "TPS2116 provides static source isolation; no supply transfer occurs during a test."
- note removed: "U1001 - TPS2116 Power Mux with Manual and Priority Switchover"
- note removed: "U1001 - TPS22917 Ultra-Low Leakage Load Switch"
- note removed: "U1001 selects the ROUTING_LOGIC_3V3 source: OFF -> output disabled STANDALONE -> TI_TARGET_3V3 STANDALONE EXT -> EXT_3V3 SUPERVISOR -> EXT_3V3"
- note removed: "U1002 - TPS22917DBV Active-high Test Block 3.3 V load switch. C1005 controls turn-on slew and inrush current. QOD discharges TEST_BLOCK_3V3 when disabled. No current limiting or overload protection."
- note removed: "| Device| OR inputs | Output | | |-------|---------------------------------------------|------------------------|-----------------------------------------------------------------------------------| | D1001 | MODE_STANDALONE_EXT , MODE_SUPERVISOR | MODE_EXT_SELECTED | Indicates that U1001 must use the external 3.3 V supply. | | D1002 | MODE_STANDALONE , MODE_EXT_SELECTED | MUX_MODE | Enables U1001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"
- moved on the sheet: C1004, C1005, D1005, R1004
