File: KICAD/V2/RevA/Espruino_Harness_RevA/routing_control.kicad_sch (KiCad schematic)
At the start: 76 parts, among them U601 TMUX1511, U602 TMUX1511, U603 TMUX1511, U604 TMUX1511, U605 TMUX1511, U606 TMUX1511, U607 TPS3808G30DBVR, U608 TPS3808G30DBVR, U609 TPS3808G30DBVR, U610 MCP23017-E/SO RCTRL0, U611 MCP23017-E/SO RCTRL1

Commit message: Implement RC01 routing baseline metadata
Parts:
- removed R13, R18, R23, R25, R603, R608: 100k, Resistor_SMD:R_0603_1608Metric, symbol Device:R
- C601, C602, C603, C604, C605, C606, C607, C608, C609, C610, C611: AISLER_MPN (none) -> 100nF 10% 16V X7R 0603
- R11, R12, R14, R15, R16, R17, R19, R20, R21, R22, R24, R601, R602, R604, R605, R606, R607, R609, R610: AISLER_MPN (none) -> 100k 0603 1% 0.1W
- TP601, TP602, TP603, TP604, TP605, TP606, TP607, TP608, TP609, TP610, TP611, TP612, TP613, TP614: MPN (none) -> 61300111121; now not fitted
- U601, U602, U603, U604, U605, U606: MPN (none) -> TMUX1511PWR
Other:
- note added: "(commands ->; controller readback <-)"
- note added: "->"
- note added: "<->"
- note added: "CONTROL AND SIGNAL-PATH FLOW SUMMARY"
- note added: "CONTROL-PLANE ISOLATION AND STARTUP - FIXED I2C BOUNDARIES AND HARDWARE CLEAR"
- note added: "HARDWARE SAFE STATE ROUTE_CLEAR_N resets both controllers; 100k pull-downs then hold every RP enable low. With ROUTING_LOGIC_3V3 absent, TMUX1511 signal paths remain Hi-Z for 0V to 3.6V."
- note added: "POWER-QUALIFIED ISOLATION AND STARTUP U606 IP01/IP02: Target I2C <-> ROUTE_I2C U606 IP03/IP04: ROUTE_I2C <-> Test Block I2C U607: qualifies the IP01/IP02 enable U608: qualifies the IP03/IP04 enable U609: qualifies ROUTE_CLEAR_N for U610/U611"
- note added: "ROUTE_I2C_SDA / ROUTE_I2C_SCL"
- note added: "ROUTING CONTROLLERS - TARGET-OWNED I2C CONTROL AND READBACK"
- note added: "ROUTING CONTROLLERS U610 / RCTRL0 / 0x21: RP01-RP16 U611 / RCTRL1 / 0x22: RP17-RP19"
- note added: "ROUTING FABRIC - 19 INDEPENDENT TARGET-TO-TEST-BLOCK PATHS"
- note added: "RP01_EN-RP19_EN ↓ ROUTING FABRIC U601-U605: RP01-RP19 ↓ NAMED TI_* TEST BLOCK ENDPOINTS ADDITIONAL U611 CONTROL BRANCH UP01_EN-UP04_EN -> U701, TB07 UART switching"
- note added: "SAFE ROUTE CHANGE One destination maximum per R0-R6 entry. Disable drivers -> clear and verify old routes -> select and verify new routes -> enable drivers."
- note added: "SWITCH FUNCTION Each TMUX1511 channel is bidirectional. EN=1 joins one R0-R6 entry to its named TI_* endpoint; EN=0 isolates it."
- note added: "TARGET FIRMWARE — TARGET-OWNED DIRECT I2C TI_I2C_SDA / TI_I2C_SCL"
- note removed: "100k on every RP control; TMUX1511 internal 6M pull-downs provide additional bias"
- note removed: "EXTERNAL SAFE-STATE PULL-DOWNS"
- note removed: "Each route entry is one-hot; every path defaults open"
- note removed: "FIXED I2C POWER-DOMAIN ISOLATION"
- note removed: "ROUTING CONTROL — DIRECT TARGET I2C, ADDRESSES 0x21 / 0x22"
- note removed: "ROUTING FABRIC — 19 ACCEPTED ROUTE-SELECTION PATHS"
- moved on the sheet: C601, C602, C603, C604, C605, C606, C607, C608, C609, C610, C611, JP610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

Commit message: Verify RC02 routing control baseline
Add the qualified fixed-I2C isolation and Hardware Clear implementation, exact component metadata, deterministic RC02 connectivity contract, accepted ERC/connectivity evidence, and visual review records. Synchronize the draft PCB and document the PCB-stage workflow while preserving the verified RC01 baseline.
Parts:
- added C621, C622, C623: 4.7nF, Capacitor_SMD:C_0603_1608Metric, symbol Device:C
- JP613: value A0 default 1 -> A0 default 0
- JP614: value A1 default 0 -> A1 default 1
- U607, U608, U609: MPN (none) -> TPS3808G30DBVR
- U610, U611: MPN (none) -> MCP23017-E/SO
Connections:
- net ROUTING_LOGIC_3V3: now also C623.1
- net TEST_BLOCK_3V3: now also C622.1
- net TI_GND: now also C621.2, C622.2, C623.2
- net TI_TARGET_3V3: now also C621.1
Other:
- moved on the sheet: C607, C608, C609, R630, R631, TP609, TP610, TP614, U607
