File: KICAD/V2/RevA/DaughterBoards/DB-ESPRUINO-CORE-GRID/DB-ESPRUINO-CORE-GRID.kicad_pcb (KiCad board)
At the start: 2 copper layers, 85.9 x 90 mm, 5 parts, among them J900 TARGET INTERFACE CONNECTOR A, J901 TARGET INTERFACE CONNECTOR B

Commit message: Implement Rev-A daughter-board foundations
Parts:
- EXT1, EXT2: footprint GenericDaughterBoardV1:HN1x22 -> V2_DaughterBoard_Targets:HN1x22
- U$1: footprint GenericDaughterBoardV1:ESPRUINO_PICO_SMD -> V2_DaughterBoard_Targets:ESPRUINO_PICO_SMD
Changed lines of the file:
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@@
 	(net 99 "/TI_ONEWIRE_DQ")
 	(net 100 "/TI_ONEWIRE_GPIO_B_FB")
-	(footprint "GenericDaughterBoardV1:HN1x22"
+	(footprint "V2_DaughterBoard_Targets:HN1x22"
 		(layer "F.Cu")
 		(at 203.623414 87.63 -90)
@@
 		)
 		(sheetname "/")
-		(sheetfile "GenericDaughterBoardV1.kicad_sch")
+		(sheetfile "DB-ESPRUINO-CORE-GRID.kicad_sch")
 		(solder_mask_margin 0.0508)
 		(solder_paste_margin -0.0508)
@@
 		)
 	)
-	(footprint "GenericDaughterBoardV1:ESPRUINO_PICO_SMD"
+	(footprint "V2_DaughterBoard_Targets:ESPRUINO_PICO_SMD"
 		(layer "F.Cu")
 		(at 189.653414 90.17 90)
@@
 		)
 		(sheetname "/")
-		(sheetfile "GenericDaughterBoardV1.kicad_sch")
+		(sheetfile "DB-ESPRUINO-CORE-GRID.kicad_sch")
 		(fp_line
 			(start 7.62 -7.62)
@@
 		(embedded_fonts no)
 	)
-	(footprint "GenericDaughterBoardV1:HN1x22"
+	(footprint "V2_DaughterBoard_Targets:HN1x22"
 		(layer "F.Cu")
 		(at 178.223414 87.63 -90)
@@
 		)
 		(sheetname "/")
-		(sheetfile "GenericDaughterBoardV1.kicad_sch")
+		(sheetfile "DB-ESPRUINO-CORE-GRID.kicad_sch")
 		(solder_mask_margin 0.0508)
 		(solder_paste_margin -0.0508)
@@
 		(property ki_fp_filters "Connector*:*_2x12_*")
 		(sheetname "/")
-		(sheetfile "GenericDaughterBoardV1.kicad_sch")
+		(sheetfile "DB-ESPRUINO-CORE-GRID.kicad_sch")
 		(attr through_hole)
 		(fp_line
@@
 		(property ki_fp_filters "Connector*:*_2x12_*")
 		(sheetname "/")
-		(sheetfile "GenericDaughterBoardV1.kicad_sch")
+		(sheetfile "DB-ESPRUINO-CORE-GRID.kicad_sch")
 		(attr through_hole)
 		(fp_line
