File: KICAD/V2/RevA/DaughterBoards/DB-PICO-XIAO-GRID/DB-PICO-XIAO-GRID.kicad_sch (KiCad schematic)
At the start: 5 parts, among them J900 TARGET INTERFACE CONNECTOR A, J901 TARGET INTERFACE CONNECTOR B

Commit message: Implement Rev-A daughter-board foundations
Parts:
- EXT1, EXT2: footprint GenericDaughterBoardV1:HN1x22 -> V2_DaughterBoard_Targets:HN1x22; symbol GenericDaughterBoardV1:CON22 -> V2_DaughterBoard_Targets:CON22
- J900, J901: footprint Connector_PinHeader_2.54mm:PinHeader_2x12_P2.54mm_Vertical -> V2_Target_Interface:TargetInterface_2x12_P2.54mm_RA_Male_Adafruit1541_Daughter; symbol GenericDaughterBoardV1:Target_Interface_2x12_Odd_Even -> V2_DaughterBoard_Targets:Target_Interface_2x12_Odd_Even
- U$1: footprint GenericDaughterBoardV1:ESPRUINO_PICO_SMD -> V2_DaughterBoard_Targets:ESPRUINO_PICO_SMD; symbol GenericDaughterBoardV1:ESPRUINO_PICO_SMD -> V2_DaughterBoard_Targets:ESPRUINO_PICO_SMD
Changed lines of the file:
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@@
 		)
 		(instances
-			(project "GenericDaughterBoardV1"
+			(project "DB-PICO-XIAO-GRID"
 				(path "/f947ec4c-e81e-4f1c-bec8-b3723a2b92bb"
 					(reference "#PWR04")
@@
 		)
 		(instances
-			(project "GenericDaughterBoardV1"
+			(project "DB-PICO-XIAO-GRID"
 				(path "/f947ec4c-e81e-4f1c-bec8-b3723a2b92bb"
 					(reference "#PWR07")
@@
 		)
 		(instances
-			(project "GenericDaughterBoardV1"
+			(project "DB-PICO-XIAO-GRID"
 				(path "/f947ec4c-e81e-4f1c-bec8-b3723a2b92bb"
 					(reference "#PWR06")
@@
 		)
 		(instances
-			(project "GenericDaughterBoardV1"
+			(project "DB-PICO-XIAO-GRID"
 				(path "/f947ec4c-e81e-4f1c-bec8-b3723a2b92bb"
 					(reference "#PWR024")
@@
 		)
 		(instances
-			(project "GenericDaughterBoardV1"
+			(project "DB-PICO-XIAO-GRID"
 				(path "/f947ec4c-e81e-4f1c-bec8-b3723a2b92bb"
 					(reference "#PWR023")
@@
 	)
 	(symbol
-		(lib_id "GenericDaughterBoardV1:CON22")
+		(lib_id "V2_DaughterBoard_Targets:CON22")
 		(at 257.81 180.34 0)
 		(mirror y)
@@
 			)
 		)
-		(property "Footprint" "GenericDaughterBoardV1:HN1x22"
+		(property "Footprint" "V2_DaughterBoard_Targets:HN1x22"
 			(at 257.175 212.09 0)
 			(effects
@@
 		)
 		(instances
-			(project "GenericDaughterBoardV1"
+			(project "DB-PICO-XIAO-GRID"
 				(path "/f947ec4c-e81e-4f1c-bec8-b3723a2b92bb"
 					(reference "EXT1")
@@
 	)
 	(symbol
-		(lib_id "GenericDaughterBoardV1:CON22")
+		(lib_id "V2_DaughterBoard_Targets:CON22")
 		(at 287.02 180.34 0)
 		(unit 1)
@@
 			)
 		)
-		(property "Footprint" "GenericDaughterBoardV1:HN1x22"
+		(property "Footprint" "V2_DaughterBoard_Targets:HN1x22"
 			(at 287.655 212.09 0)
 			(effects
@@
 		)
 		(instances
-			(project "GenericDaughterBoardV1"
+			(project "DB-PICO-XIAO-GRID"
 				(path "/f947ec4c-e81e-4f1c-bec8-b3723a2b92bb"
 					(reference "EXT2")
@@
 		)
 		(instances
-			(project "GenericDaughterBoardV1"
+			(project "DB-PICO-XIAO-GRID"
 				(path "/f947ec4c-e81e-4f1c-bec8-b3723a2b92bb"
 					(reference "#PWR05")
@@
 	(symbol
 		(lib_name "Target_Interface_2x12_Odd_Even_1")
-		(lib_id "GenericDaughterBoardV1:Target_Interface_2x12_Odd_Even")
+		(lib_id "V2_DaughterBoard_Targets:Target_Interface_2x12_Odd_Even")
 		(at 119.38 88.9 0)
 		(unit 1)
@@
 			)
 		)
-		(property "Footprint" "Connector_PinHeader_2.54mm:PinHeader_2x12_P2.54mm_Vertical"
+		(property "Footprint" "V2_Target_Interface:TargetInterface_2x12_P2.54mm_RA_Male_Adafruit1541_Daughter"
 			(at 119.38 88.9 0)
 			(effects
@@
 		)
 		(instances
-			(project "GenericDaughterBoardV1"
+			(project "DB-PICO-XIAO-GRID"
 				(path "/f947ec4c-e81e-4f1c-bec8-b3723a2b92bb"
 					(reference "J900")
@@
 	)
 	(symbol
-		(lib_id "GenericDaughterBoardV1:ESPRUINO_PICO_SMD")
+		(lib_id "V2_DaughterBoard_Targets:ESPRUINO_PICO_SMD")
 		(at 281.94 67.31 0)
 		(unit 1)
@@
 			)
 		)
-		(property "Footprint" "GenericDaughterBoardV1:ESPRUINO_PICO_SMD"
+		(property "Footprint" "V2_DaughterBoard_Targets:ESPRUINO_PICO_SMD"
 			(at 281.94 67.31 0)
 			(effects
@@
 		)
 		(instances
-			(project "GenericDaughterBoardV1"
+			(project "DB-PICO-XIAO-GRID"
 				(path "/f947ec4c-e81e-4f1c-bec8-b3723a2b92bb"
 					(reference "U$1")
@@
 		)
 		(instances
-			(project "GenericDaughterBoardV1"
+			(project "DB-PICO-XIAO-GRID"
 				(path "/f947ec4c-e81e-4f1c-bec8-b3723a2b92bb"
 					(reference "#FLG03")
@@
 		)
 		(instances
-			(project "GenericDaughterBoardV1"
+			(project "DB-PICO-XIAO-GRID"
 				(path "/f947ec4c-e81e-4f1c-bec8-b3723a2b92bb"
 					(reference "#FLG01")
@@
 	)
 	(symbol
-		(lib_id "GenericDaughterBoardV1:Target_Interface_2x12_Odd_Even")
+		(lib_id "V2_DaughterBoard_Targets:Target_Interface_2x12_Odd_Even")
 		(at 119.38 168.91 0)
 		(unit 1)
@@
 			)
 		)
-		(property "Footprint" "Connector_PinHeader_2.54mm:PinHeader_2x12_P2.54mm_Vertical"
+		(property "Footprint" "V2_Target_Interface:TargetInterface_2x12_P2.54mm_RA_Male_Adafruit1541_Daughter"
 			(at 119.38 168.91 0)
 			(effects
@@
 		)
 		(instances
-			(project "GenericDaughterBoardV1"
+			(project "DB-PICO-XIAO-GRID"
 				(path "/f947ec4c-e81e-4f1c-bec8-b3723a2b92bb"
 					(reference "J901")
